Commit message: init sentry

File: Main_ws/src/rm_robot_description/urdf/rm_gimbal.urdf.xacro (robot description, xacro)
@@ -5,13 +5,13 @@
   <xacro:arg name="rpy" default="0 0 0" />
   <link name="odom" />
-  <link name="gimbal_link" />
+  <link name="gimbal_link_aim" />
   <joint name="gimbal_joint" type="floating">
     <parent link="odom" />
-    <child link="gimbal_link" />
+    <child link="gimbal_link_aim" />
   </joint>
   <link name="camera_link" />
   <joint name="camera_joint" type="fixed">
     <origin xyz="$(arg xyz)" rpy="$(arg rpy)" />
-    <parent link="gimbal_link" />
+    <parent link="gimbal_link_aim" />
     <child link="camera_link" />
     <axis xyz="0 0 0" />
